File: hardware/rf_controller.sch (KiCad schematic (older format))
At the start: 32 parts

Commit message: + Add pcb
Parts:
- C1, C10, C11, C12, C2, C3, C4, C5, C6, C7, C8, C9: renamed from C?; footprint CAP_0603 -> Capacitors:CAP_0603
- D1: renamed from D?; footprint (none) -> Diodes:SOD323
- DA1: renamed from DA?; footprint (none) -> TO_SOT_Packages_SMD:SOT-23-5_HandSoldering
- DD1: renamed from DD?; footprint (none) -> Housings_DFN_QFN:QFN-32-1EP_5x5mm_Pitch0.5mm
- L1: renamed from L?; footprint (none) -> Inductors:CD_type_6.0X5.5
- R1, R2, R3, R4, R5: renamed from R?; footprint RES_0603 -> Capacitors:CAP_0603
- SW1: renamed from SW?; footprint (none) -> BtnsSwitches:SW_SS-1P2T
- SW2, SW3, SW4: renamed from SW?; footprint (none) -> BtnsSwitches:PUSH_THRHOLE_3-1825910-5
- U1: renamed from U?; footprint (none) -> BtnsSwitches:ENC_E11X
- XL1, XL3: renamed from XL?; footprint (none) -> Connectors:PLS-2
- XL2: renamed from XL?; footprint (none) -> Installation:CC1101_MODULE
- XL4: renamed from XL?; footprint (none) -> Display:84x48_LCD_Module
- XL5: renamed from XL?; footprint (none) -> Connectors:PLS-4
- XL6: renamed from XL?; footprint (none) -> Connectors:PLS-3
Connections:
- net СС1101_SCK is gone; now on net CC1101_CLK: XL2.4

Commit message: + Add FW project; + Add HW gerber files.
Parts:
- R1, R2, R3, R4, R5: footprint Capacitors:CAP_0603 -> Resistors:RES_0603
- SW2: value BUTTON -> BUTTON1
- SW3: value BUTTON -> BUTTON2
- SW4: value BUTTON -> BUTTON3/RST
- XL1: footprint Connectors:PLS-2 -> Installation:2xBAT_AA_SOLDER
Connections:
- net BAT: now reaches SW1.1, XL1.2 (PM)
- net PWR_IN: now reaches D1.A, DA1.5 (LX), L1.1
Changed lines of the file:
@@
 F 0 "XL1" V 850 6350 40  0000 C CNN
 F 1 "CONN_2" V 950 6350 40  0000 C CNN
-F 2 "Connectors:PLS-2" H 900 6350 60  0001 C CNN
+F 2 "Installation:2xBAT_AA_SOLDER" H 900 6350 60  0001 C CNN
 F 3 "" H 900 6350 60  0000 C CNN
 	1    900  6350
@@
 F 0 "R2" V 5630 5750 50  0000 C CNN
 F 1 "10k" V 5550 5900 50  0000 C CNN
-F 2 "Capacitors:CAP_0603" V 5630 6000 28  0000 C CNN
+F 2 "Resistors:RES_0603" V 5630 6000 28  0000 C CNN
 F 3 "" H 5550 5900 60  0000 C CNN
 	1    5550 5900
@@
 F 0 "R3" V 5630 6450 50  0000 C CNN
 F 1 "10k" V 5550 6600 50  0000 C CNN
-F 2 "Capacitors:CAP_0603" V 5630 6700 28  0000 C CNN
+F 2 "Resistors:RES_0603" V 5630 6700 28  0000 C CNN
 F 3 "" H 5550 6600 60  0000 C CNN
 	1    5550 6600
@@
 P 9250 3250
 F 0 "SW2" H 9050 3400 50  0000 C CNN
-F 1 "BUTTON" H 9350 3400 50  0000 C CNN
+F 1 "BUTTON1" H 9350 3400 50  0000 C CNN
 F 2 "BtnsSwitches:PUSH_THRHOLE_3-1825910-5" H 9250 3250 60  0001 C CNN
 F 3 "" H 9250 3250 60  0000 C CNN
@@
 P 9250 3550
 F 0 "SW3" H 9050 3700 50  0000 C CNN
-F 1 "BUTTON" H 9350 3700 50  0000 C CNN
+F 1 "BUTTON2" H 9350 3700 50  0000 C CNN
 F 2 "BtnsSwitches:PUSH_THRHOLE_3-1825910-5" H 9250 3550 60  0001 C CNN
 F 3 "" H 9250 3550 60  0000 C CNN
@@
 U 1 1 5BC9DA11
 P 9250 3850
-F 0 "SW4" H 9050 4000 50  0000 C CNN
-F 1 "BUTTON" H 9350 4000 50  0000 C CNN
+F 0 "SW4" H 8950 4000 50  0000 C CNN
+F 1 "BUTTON3/RST" H 9350 4000 50  0000 C CNN
 F 2 "BtnsSwitches:PUSH_THRHOLE_3-1825910-5" H 9250 3850 60  0001 C CNN
 F 3 "" H 9250 3850 60  0000 C CNN
@@
 F 0 "R1" V 4030 1300 50  0000 C CNN
 F 1 "10k" V 3950 1450 50  0000 C CNN
-F 2 "Capacitors:CAP_0603" V 4030 1550 28  0000 C CNN
+F 2 "Resistors:RES_0603" V 4030 1550 28  0000 C CNN
 F 3 "" H 3950 1450 60  0000 C CNN
 	1    3950 1450
@@
 F 0 "R4" V 9080 1250 50  0000 C CNN
 F 1 "10k" V 9000 1400 50  0000 C CNN
-F 2 "Capacitors:CAP_0603" V 9080 1500 28  0000 C CNN
+F 2 "Resistors:RES_0603" V 9080 1500 28  0000 C CNN
 F 3 "" H 9000 1400 60  0000 C CNN
 	1    9000 1400
@@
 F 0 "R5" V 9580 1250 50  0000 C CNN
 F 1 "10k" V 9500 1400 50  0000 C CNN
-F 2 "Capacitors:CAP_0603" V 9580 1500 28  0000 C CNN
+F 2 "Resistors:RES_0603" V 9580 1500 28  0000 C CNN
 F 3 "" H 9500 1400 60  0000 C CNN
 	1    9500 1400
@@
 	8850 2000 9650 2000
 Connection ~ 9500 2000
+Text Label 1150 6250 0    60   ~ 0
+BAT
+Text Label 3050 5900 0    60   ~ 0
+PWR_IN
 $EndSCHEMATC
